File: Kicad/incubator/LCD_16x2.sch (KiCad schematic (older format))
At the start: 6 parts, among them SW2 Rotary_Encoder_Switch

Commit message: fix: fan size and push button position
Parts:
- DS1: symbol Display_Character:WC1602A -> incubator-rescue:WC1602A-Display_Character
- R6, R7, R8: symbol Device:R -> incubator-rescue:R-Device
- RV1: symbol Device:R_POT -> incubator-rescue:R_POT-Device
- SW2: symbol Device:Rotary_Encoder_Switch -> incubator-rescue:Rotary_Encoder_Switch-Device
Changed lines of the file:
@@
 	6875 4750 6875 4650
 $Comp
-L power:GND #PWR?
+L incubator-rescue:GND-power #PWR?
 U 1 1 611BC109
 P 6875 4750
@@
 	6200 4550 6125 4550
 $Comp
-L power:GND #PWR?
+L incubator-rescue:GND-power #PWR?
 U 1 1 611BC115
 P 6125 4750
@@
 $EndComp
 $Comp
-L Device:R_POT RV?
+L incubator-rescue:R_POT-Device RV?
 U 1 1 611BC11B
 P 6825 3175
@@
 	4925 3450 4925 3275
 $Comp
-L power:GND #PWR?
+L incubator-rescue:GND-power #PWR?
 U 1 1 611BC128
 P 4925 3450
@@
 	5800 3575 5875 3575
 $Comp
-L power:GND #PWR?
+L incubator-rescue:GND-power #PWR?
 U 1 1 611BC13D
 P 5875 3625
@@
 	6825 3825 6825 3725
 $Comp
-L power:GND #PWR?
+L incubator-rescue:GND-power #PWR?
 U 1 1 611BC148
 P 6825 3825
@@
 $EndComp
 $Comp
-L Device:R R?
+L incubator-rescue:R-Device R?
 U 1 1 611BC14E
 P 6825 2775
@@
 $EndComp
 $Comp
-L Device:R R?
+L incubator-rescue:R-Device R?
 U 1 1 611BC154
 P 6825 3575
@@
 $EndComp
 $Comp
-L Device:R R?
+L incubator-rescue:R-Device R?
 U 1 1 611BC15A
 P 6050 3475
@@
 $EndComp
 $Comp
-L Device:Rotary_Encoder_Switch SW?
+L incubator-rescue:Rotary_Encoder_Switch-Device SW?
 U 1 1 611BC160
 P 6500 4550
@@
 $EndComp
 $Comp
-L Display_Character:WC1602A DS?
+L incubator-rescue:WC1602A-Display_Character DS?
 U 1 1 611BC166
 P 5400 3775
@@
 D7
 $Comp
-L power:GND #PWR?
+L incubator-rescue:GND-power #PWR?
 U 1 1 611BFC11
 P 5400 4700
