File: kicad/simple-i2c-screen/atmega328p.sch (KiCad schematic (older format))
At the start: 5 parts, among them U2 ATmega328P-AU

Commit message: refactor: version 1.0.3 for PCB change MOITORING_LED to pin 13 like Arduino
Connections:
- net B7: no longer names the net of U2.8 (XTAL2/PB7)
- no-connect marks 6 -> 7
Changed lines of the file:
@@
 $Descr A4 11693 8268
 encoding utf-8
-Sheet 3 3
+Sheet 2 3
 Title ""
 Date ""
@@
 Text HLabel 7050 2750 2    50   Input ~ 0
 B6
-Text HLabel 7050 2850 2    50   Input ~ 0
-B7
 Wire Wire Line
 	6350 4850 6350 4950
@@
 NoConn ~ 6950 2250
 NoConn ~ 6950 2350
-Wire Wire Line
-	6950 2850 7050 2850
 Wire Wire Line
 	7050 2750 6950 2750
@@
 Wire Wire Line
 	7050 4550 6950 4550
+NoConn ~ 6950 2850
 $EndSCHEMATC
